Commit message: added random containers with colors

File: cliport/environments/assets/block/block.urdf (robot description, URDF)
Before this commit: robot box.urdf, 1 links, 0 joints
Links:
- link baseLink: geometry collision box size=0.04 0.04 0.04; visual box size=0.1 0.1 0.1

File: cliport/environments/assets/bowl/bowl.urdf (robot description, URDF)
Before this commit: robot bowl.urdf, 1 links, 0 joints
Links:
- link baseLink: geometry collision mesh filename=cup.obj scale=1.25 1.25 0.25; visual mesh filename=textured-0008192.obj scale=2.5 2.5 0.5
